File: KiCAD/BeagleBone Black Cape/BBB-Cape.sch (KiCad schematic (older format))
At the start: 8 parts, among them J1 MOUNTING_HOLE, J2 MOUNTING_HOLE, J3 MOUNTING_HOLE, J4 MOUNTING_HOLE, J5 MOUNTING_HOLE, J6 MOUNTING_HOLE, J7 MOUNTING_HOLE, J8 MOUNTING_HOLE

Commit message: BeagleBone Updated, headers need to be moved into proper spot
Parts:
- removed J5, J6, J7, J8: MOUNTING_HOLE, Mounting_Holes:MountingHole_3.2mm_M3_Pad, symbol MOUNTING_HOLE
Other:
- note added: "Index:\n\nPins and Connectors.............................Page 1\n\n"
- note removed: "1\n"
- note removed: "BBB-Socket"
- note removed: "Index"
- note removed: "Index:\n\nPins and Connectors.............................Page 1\nRJ45 and WIZnet W5500.......................Page 2\nBuck Reg...............................................Page 3\nRS485....................................................Page 4\n\n"
- note removed: "Mitchell Stride & Mark Belbin\n"
- note removed: "Nov. 10/2017"
- note removed: "PARADIGM HYPERLOOP"
